Commit message: SH industry and gripper franka update

File: model/calibrator_softhand_industry.urdf.xacro (robot description, xacro)
@@ -1,5 +1,5 @@
 <?xml version="1.0"?>
 <robot xmlns:xacro="http://www.ros.org/wiki/xacro">
-<xacro:macro name="calibrator_pandagripper" params="parent name *origin">
+<xacro:macro name="calibrator_softhand_industry" params="parent name *origin">
   <joint name="${parent}_${name}_base_joint" type="fixed">
     <xacro:insert_block name="origin"/>
@@ -23,6 +23,6 @@
   <joint name="${name}_joint" type="fixed">
 <!--     <origin xyz="-0.04 0 0" rpy="0 0 1.57079633"/>-->
-    <origin xyz="-0.025279067 0.025279067 0.028500000" rpy="0 -1.5708 -0.7853982"/>
-    <!-- <origin xyz="-0.025279067 0.025279067 0.028500000" rpy="-1.5708 -0.7853982 1.5708"/> -->
+    <!-- <origin xyz="-0.019884 0 0.02868" rpy="0.5235989 0 1.5707963"/> -->
+    <origin xyz="0.0 -0.044 0.022" rpy="1.5707963 0.0 0.0"/>
     <parent link="${name}_mesh"/>
     <child link="${name}"/>

Commit message: update gofa calib

File: model/calibrator_softhand_industry.urdf.xacro (robot description, xacro)
@@ -22,7 +22,6 @@
   <!-- this is where the ar marker is w.r.t. the mesh, known from CAD model -->
   <joint name="${name}_joint" type="fixed">
-<!--     <origin xyz="-0.04 0 0" rpy="0 0 1.57079633"/>-->
-    <!-- <origin xyz="-0.019884 0 0.02868" rpy="0.5235989 0 1.5707963"/> -->
-    <origin xyz="0.0 -0.044 0.022" rpy="1.5707963 0.0 0.0"/>
+    <!-- <origin xyz="0.0 -0.044 0.022" rpy="1.5707963 0.0 0.0"/> Franka -->
+    <origin xyz="0.0546 0.044 0.0" rpy="-1.5707963 0.0 0.0"/> <!--GOFA -->
     <parent link="${name}_mesh"/>
     <child link="${name}"/>

File: robots/gofa_arm_SH_industry_calibration.urdf.xacro (robot description, xacro)
@@ -1,5 +1,5 @@
 <?xml version='1.0' encoding='utf-8'?>
 <robot xmlns:xacro="http://www.ros.org/wiki/xacro" name="gofa">
-  <xacro:include filename="$(find gofa_description)/urdf/gofa.urdf" />
+  <xacro:include filename="$(find gofa_description)/urdf/gofa.urdf.xacro" />
   <xacro:include filename="$(find calibration)/model/calibrator_softhand_industry.urdf.xacro"/>
   <xacro:gofa />

Commit message: update

File: model/calibrator_softhand_industry.urdf.xacro (robot description, xacro)
@@ -23,5 +23,5 @@
   <joint name="${name}_joint" type="fixed">
     <!-- <origin xyz="0.0 -0.044 0.022" rpy="1.5707963 0.0 0.0"/> Franka -->
-    <origin xyz="0.0546 0.044 0.0" rpy="-1.5707963 0.0 0.0"/> <!--GOFA -->
+    <origin xyz="0.0546 0.044 0.0" rpy="-1.5707963 0.0 -1.5707963"/> <!--GOFA -->
     <parent link="${name}_mesh"/>
     <child link="${name}"/>

Commit message: update

File: model/calibrator_softhand_industry.urdf.xacro (robot description, xacro)
@@ -23,5 +23,5 @@
   <joint name="${name}_joint" type="fixed">
     <!-- <origin xyz="0.0 -0.044 0.022" rpy="1.5707963 0.0 0.0"/> Franka -->
-    <origin xyz="0.0546 0.044 0.0" rpy="-1.5707963 0.0 -1.5707963"/> <!--GOFA -->
+    <origin xyz="0.0546 0.044 0.0" rpy="0.0 -1.5707963 -1.5707963"/> <!--GOFA -->
     <parent link="${name}_mesh"/>
     <child link="${name}"/>

Commit message: update

File: model/calibrator_softhand_industry.urdf.xacro (robot description, xacro)
@@ -8,20 +8,15 @@
   </joint>
   <link name="${name}_mesh">
-<!--     <visual>
+    <visual>
       <geometry>
-        <mesh filename="package://franka_description/meshes/camera_robot_calibrator.stl"/>
+        <mesh filename="package://calibration/resources/3DPrints/qb_industry_target_v01.dae" scale="0.001 0.001 0.001"/>
       </geometry>
       <material name="Vito/Silver"/>
     </visual>
-    <collision>
-      <geometry>
-        <mesh filename="package://franka_description/meshes/camera_robot_calibrator.stl"/>
-      </geometry>
-    </collision> -->
   </link>
   <!-- this is where the ar marker is w.r.t. the mesh, known from CAD model -->
   <joint name="${name}_joint" type="fixed">
     <!-- <origin xyz="0.0 -0.044 0.022" rpy="1.5707963 0.0 0.0"/> Franka -->
-    <origin xyz="0.0546 0.044 0.0" rpy="0.0 -1.5707963 -1.5707963"/> <!--GOFA -->
+    <origin xyz="0 0.0285 -0.044" rpy="0 3.141592 0"/><!--GOFA-->
     <parent link="${name}_mesh"/>
     <child link="${name}"/>

File: robots/gofa_arm_SH_industry_calibration.urdf.xacro (robot description, xacro)
@@ -6,5 +6,5 @@
   <!-- from the CAD model, the frame coincides with the 7-th link -->
   <xacro:calibrator_softhand_industry name="calibrator_softhand_industry" parent="tool0">
-    <origin xyz="0 0 0" rpy="0 0 0"/>
+    <origin xyz="-0.0065 0 0" rpy="1.5707963 1.5707963 0"/> <!-- il frame della mesh del calibrator è sulla superfice esterna -->
   </xacro:calibrator_softhand_industry>
 </robot>

Commit message: update

File: model/calibrator_softhand_industry.urdf.xacro (robot description, xacro)
@@ -17,6 +17,5 @@
   <!-- this is where the ar marker is w.r.t. the mesh, known from CAD model -->
   <joint name="${name}_joint" type="fixed">
-    <!-- <origin xyz="0.0 -0.044 0.022" rpy="1.5707963 0.0 0.0"/> Franka -->
-    <origin xyz="0 0.0285 -0.044" rpy="0 3.141592 0"/><!--GOFA-->
+      <origin xyz="0 0.0285 -0.044" rpy="0 3.141592 0"/>
     <parent link="${name}_mesh"/>
     <child link="${name}"/>

File: robots/panda_arm_SH_industry_calibration.urdf.xacro (robot description, xacro)
@@ -6,5 +6,5 @@
   <!-- from the CAD model, the frame coincides with the 7-th link -->
   <xacro:calibrator_softhand_industry name="calibrator_softhand_industry" parent="panda_link8">
-    <origin xyz="0 0 0" rpy="0 0 0"/>
+    <origin xyz="0 0 -0.0065" rpy="1.5707963 0.0 3.141592"/>
   </xacro:calibrator_softhand_industry>
 </robot>

Commit message: update

File: model/calibrator_softhand_industry.urdf.xacro (robot description, xacro)
@@ -10,5 +10,5 @@
     <visual>
       <geometry>
-        <mesh filename="package://calibration/resources/3DPrints/qb_industry_target_v01.dae" scale="0.001 0.001 0.001"/>
+        <mesh filename="package://calibration/resources/3DPrints/flange_target.dae" scale="0.001 0.001 0.001"/>
       </geometry>
       <material name="Vito/Silver"/>
@@ -17,5 +17,6 @@
   <!-- this is where the ar marker is w.r.t. the mesh, known from CAD model -->
   <joint name="${name}_joint" type="fixed">
-      <origin xyz="0 0.0285 -0.044" rpy="0 3.141592 0"/>
+      <!-- <origin xyz="0 0.0285 -0.044" rpy="0 3.141592 0"/> -->
+      <origin xyz="0.0445 0.031  0" rpy="0 1.5707963 0"/>
     <parent link="${name}_mesh"/>
     <child link="${name}"/>

File: robots/gofa_arm_SH_industry_calibration.urdf.xacro (robot description, xacro)
@@ -6,5 +6,6 @@
   <!-- from the CAD model, the frame coincides with the 7-th link -->
   <xacro:calibrator_softhand_industry name="calibrator_softhand_industry" parent="tool0">
-    <origin xyz="-0.0065 0 0" rpy="1.5707963 1.5707963 0"/> <!-- il frame della mesh del calibrator è sulla superfice esterna -->
+    <origin xyz="-0.006 0 0" rpy=" 0 3.1415927 -1.5707963"/> <!-- il frame della mesh del calibrator è sulla superfice esterna -->
+    <!-- <origin xyz="-0.0065 0 0" rpy="1.5707963 1.5707963 0"/> da cad è questo ma in realtà no -->
   </xacro:calibrator_softhand_industry>
 </robot>

File: robots/panda_arm_SH_industry_calibration.urdf.xacro (robot description, xacro)
@@ -6,5 +6,6 @@
   <!-- from the CAD model, the frame coincides with the 7-th link -->
   <xacro:calibrator_softhand_industry name="calibrator_softhand_industry" parent="panda_link8">
-    <origin xyz="0 0 -0.0065" rpy="1.5707963 0.0 3.141592"/>
+    <origin xyz="0 0 -0.0065" rpy="1.5707963 0.0 -1.5707963"/>
+    <!-- <origin xyz="-0.006 0 0" rpy=" 0 3.1415927 -1.5707963"/> -->
   </xacro:calibrator_softhand_industry>
 </robot>
