Commit message: new calibrator

File: model/calibrator_softhand.urdf.xacro (robot description, xacro)
@@ -1,5 +1,5 @@
 <?xml version="1.0"?>
 <robot xmlns:xacro="http://www.ros.org/wiki/xacro">
-<xacro:macro name="calibrator" params="parent name *origin">
+<xacro:macro name="calibrator_softhand" params="parent name *origin">
   <joint name="${parent}_${name}_base_joint" type="fixed">
     <xacro:insert_block name="origin"/>

File: robots/panda_arm_calibration.urdf.xacro (robot description, xacro)
@@ -2,9 +2,9 @@
 <robot xmlns:xacro="http://www.ros.org/wiki/xacro" name="panda">
   <xacro:include filename="$(find franka_description)/robots/panda_arm.xacro" />
-  <xacro:include filename="$(find calibration)/model/calibrator.urdf.xacro"/>
+  <xacro:include filename="$(find calibration)/model/calibrator_pandagripper.urdf.xacro"/>
   <xacro:panda_arm />
   <!-- from the CAD model, the frame coincides with the 7-th link -->
-  <xacro:calibrator name="calibrator" parent="panda_link8">
+  <xacro:calibrator_pandagripper name="calibrator_pandagripper" parent="panda_link8">
     <origin xyz="0 0 0" rpy="0 0 0"/>
-  </xacro:calibrator>
+  </xacro:calibrator_pandagripper>
 </robot>

Commit message: update Euler angles

File: model/calibrator_softhand.urdf.xacro (robot description, xacro)
@@ -23,5 +23,6 @@
   <joint name="${name}_joint" type="fixed">
 <!--     <origin xyz="-0.04 0 0" rpy="0 0 1.57079633"/>-->
-    <origin xyz="-0.019884 0 0.02868" rpy="0.5235989 0 1.5707963"/>
+    <!-- <origin xyz="-0.019884 0 0.02868" rpy="0.5235989 0 1.5707963"/> -->
+    <origin xyz="-0.019884 0 0.02868" rpy="0.0 -1.0471972 0.0"/>
     <parent link="${name}_mesh"/>
     <child link="${name}"/>

Commit message: update

File: model/calibrator_softhand.urdf.xacro (robot description, xacro)
@@ -24,5 +24,10 @@
 <!--     <origin xyz="-0.04 0 0" rpy="0 0 1.57079633"/>-->
     <!-- <origin xyz="-0.019884 0 0.02868" rpy="0.5235989 0 1.5707963"/> -->
-    <origin xyz="-0.019884 0 0.02868" rpy="0.0 -1.0471972 0.0"/>
+    <!-- <origin xyz="-0.019884 0 0.02868" rpy="0.0 -1.0471972 0.0"/> -->
+     <!-- RIGHT ARM-->
+    <!-- <origin xyz="0.002 -0.035 0.034" rpy="0.0 -1.5707963 1.5707963"/> -->
+     <!-- LEFT ARM -->
+    <origin xyz="0.002 -0.035 0.034" rpy="0.0 -1.5707963 1.5707963"/>
+    <!-- <origin xyz="0.2 0.0 0.0" rpy="0.0 0.0 0.0"/> -->
     <parent link="${name}_mesh"/>
     <child link="${name}"/>
